Commit message: doc + hiro name

File: sig_ros/robot_desc/out.urdf (robot description, URDF)
Before this commit: robot bobby, 52 links, 51 joints
Joints:
- joint l_elbow_flex_joint: origin xyz=0.18 0 0 rpy=0 0 0 -> xyz=0.1952 0 0 rpy=0 0 0
- joint l_shoulder_pan_joint: origin xyz=0 0.168 0 rpy=0 0 0 -> xyz=0 0.1664 0 rpy=0 0 0
- joint l_wrist_flex_joint: origin xyz=0.1312 0.0 0.0 rpy=0 0 0 -> xyz=0.112 0 0 rpy=0 0 0
- joint r_elbow_flex_joint: origin xyz=0.18 0 0 rpy=0 0 0 -> xyz=0.1952 0 0 rpy=0 0 0
- joint r_shoulder_pan_joint: origin xyz=0 0.168 0 rpy=0 0 0 -> xyz=0 -0.1664 0 rpy=0 0 0
- joint r_wrist_flex_joint: origin xyz=0.1312 0.0 0.0 rpy=0 0 0 -> xyz=0.112 0 0 rpy=0 0 0
- joint torso_lift_joint: origin xyz=0 0 0.836 rpy=0 0 0 -> xyz=0 0 0.832 rpy=0 0 0

File: user/xml/out.urdf (robot description, URDF)
Before this commit: robot bobby, 52 links, 51 joints
Joints:
- joint base_footprint_joint: origin xyz=0 0 0.051 rpy=0 0 0 -> xyz=0 0 0 rpy=0 0 0
- joint l_elbow_flex_joint: origin xyz=0.4 0 0 rpy=0 0 0 -> xyz=0.0136 0.0032 -0.1952 rpy=0 0 0
- joint l_shoulder_lift_joint: origin xyz=0.1 0 0 rpy=0 0 0 -> xyz=0 0 0 rpy=0 0 0
- joint l_shoulder_pan_joint: origin xyz=0.0 0.188 0.0 rpy=0 0 0 -> xyz=-0.672 0.1664 0.832 rpy=0 0 0
- joint l_wrist_flex_joint: origin xyz=0.321 0 0 rpy=0 0 0 -> xyz=-0.02 -0.0032 -0.112 rpy=0 0 0
- joint r_elbow_flex_joint: origin xyz=0.4 0 0 rpy=0 0 0 -> xyz=0.0144 -0.0016 -0.1952 rpy=0 0 0
- joint r_shoulder_lift_joint: origin xyz=0.1 0 0 rpy=0 0 0 -> xyz=0 0 0 rpy=0 0 0
- joint r_shoulder_pan_joint: origin xyz=0.0 -0.188 0.0 rpy=0 0 0 -> xyz=-0.672 -0.1664 0.832 rpy=0 0 0
- joint r_wrist_flex_joint: origin xyz=0.321 0 0 rpy=0 0 0 -> xyz=-0.02 0.0032 -0.112 rpy=0 0 0
- joint torso_lift_joint: origin xyz=0.0 0 0.832 rpy=0 0 0 -> xyz=0 0 0.832 rpy=0 0 0
